Commit message: Add Gazebo simulation, and add dynamics in .urdf.xacro

File: install/robot_model/share/robot_model/description/robot.urdf.xacro (robot description, xacro)
@@ -32,4 +32,5 @@
         <parent link="base_link"/>
         <child link="arm_link"/>
+        <dynamics damping="0.02" friction="0.02"/>
     </joint>
     <link name = "arm_link">
@@ -51,3 +52,4 @@
         </xacro:inertial_box>
     </link>
+    <xacro:include filename="gazebo.xacro"/>
 </robot>
