Commit message: update robot model (urdf) to 3-link robot

File: install/robot_model/share/robot_model/description/gazebo.xacro (robot description, xacro)
@@ -9,6 +9,9 @@
         <material>Gazebo/Orange</material>
     </gazebo>
-    <gazebo reference="arm_link">
+    <gazebo reference="arm_link1">
         <material>Gazebo/Blue</material>
+    </gazebo>
+    <gazebo reference="arm_link2">
+        <material>Gazebo/White</material>
     </gazebo>
     <!-- Gazebo requires the use of plugins to interact with other systems such as ROS. -->

File: install/robot_model/share/robot_model/description/gazebo_ros2_control.xacro (robot description, xacro)
@@ -5,5 +5,5 @@
           <plugin>gazebo_ros2_control/GazeboSystem</plugin>
         </hardware>
-        <joint name="arm_joint">
+        <joint name="arm_joint1">
           <command_interface name="position">
             <param name="min">-10</param>
@@ -11,6 +11,8 @@
           </command_interface>
           <command_interface name = "velocity"/>
+          <command_interface name = "effort"/>
           <state_interface name="position"/>
           <state_interface name="velocity"/>
+          <state_interface name="effort"/>
         </joint>
     </ros2_control>

File: install/robot_model/share/robot_model/description/robot.urdf.xacro (robot description, xacro)
@@ -3,5 +3,4 @@
     <xacro:include filename="include.xacro" />
     <!-- This first link called "world" is empty -->
-    <!--
     <link name="world"></link>
     <joint name="base_joint" type="fixed">
@@ -10,5 +9,4 @@
         <child link="base_link"/>
     </joint>
-    -->
     <link name = "base_link">
         <visual>
@@ -29,12 +27,12 @@
         </xacro:inertial_box>
     </link>
-    <joint name="arm_joint" type = "continuous">
+    <joint name="arm_joint1" type = "continuous">
         <origin xyz = "0 0.1 0.8" rpy="${-pi/2} 0 0"/>
         <axis xyz="0.0 0.0 1.0"/>
         <parent link="base_link"/>
-        <child link="arm_link"/>
+        <child link="arm_link1"/>
         <dynamics damping="0.02" friction="0.02"/>
     </joint>
-    <link name = "arm_link">
+    <link name = "arm_link1">
         <visual>
             <origin xyz="0 0.55 0.025" rpy="${pi/2} 0 0"/>
@@ -54,4 +52,29 @@
         </xacro:inertial_box>
     </link>
+    <joint name="arm_joint2" type = "continuous">
+        <origin xyz = "0 0.9 0.05" rpy="0 0 0"/>
+        <axis xyz="0.0 0.0 1.0"/>
+        <parent link="arm_link1"/>
+        <child link="arm_link2"/>
+        <dynamics damping="0.02" friction="0.02"/>
+    </joint>
+    <link name = "arm_link2">
+        <visual>
+            <origin xyz="0 0.25 0.025" rpy="${pi/2} 0 0"/>
+            <geometry>
+                <box size="0.3 0.05 0.9"/>
+            </geometry>
+            <material name = "blue"/>
+        </visual>
+        <collision>
+            <origin xyz="0 0.25 0.025" rpy="${pi/2} 0 0"/>
+            <geometry>
+                <box size="0.3 0.05 0.9"/>
+            </geometry>
+        </collision>
+        <xacro:inertial_box mass="0.05" x="0.3" y="0.05" z="0.9">
+            <origin xyz="0 0.25 0.025" rpy="${pi/2} 0 0"/>
+        </xacro:inertial_box>
+    </link>
     <xacro:include filename="gazebo.xacro"/>
     <xacro:include filename="gazebo_ros2_control.xacro"/>
