Commit message: add my_controller2 and custom_interface pkg

File: install/robot_model/share/robot_model/description/gazebo_ros2_control.xacro (robot description, xacro)
@@ -16,9 +16,21 @@
           <state_interface name="effort"/>
         </joint>
+        <joint name="arm_joint2">
+          <command_interface name="position">
+            <param name="min">-10</param>
+            <param name="max">10</param>
+          </command_interface>
+          <command_interface name = "velocity"/>
+          <command_interface name = "effort"/>
+          <state_interface name="position"/>
+          <state_interface name="velocity"/>
+          <state_interface name="effort"/>
+        </joint>
     </ros2_control>
     <gazebo>
         <plugin name="gazebo_ros2_control" filename="libgazebo_ros2_control.so">
             <!-- <parameters>$(find robot_model)/config/my_controllers.yaml</parameters> -->
-            <parameters>$(find my_controller)/config/my_controllers_custom.yaml</parameters>
+            <!-- <parameters>$(find my_controller)/config/my_controllers_custom.yaml</parameters> -->
+            <parameters>$(find my_controller2)/config/my_controller2_custom.yaml</parameters>
         </plugin>
     </gazebo>
